File: USB tester/USB tester.kicad_sch (KiCad schematic)
At the start: 9 parts, among them J3 USB_A

Commit message: update
Parts:
- added J1: USB_A, Connector_USB:USB_A_Receptacle_GCT_USB1046, symbol Connector:USB_A
- added J2: USB_C_Receptacle_USB2.0_16P, Connector_USB:USB_C_Receptacle_G-Switch_GT-USB-7010ASV, symbol Connector:USB_C_Receptacle_USB2.0_16P
- added R10, R8, R9: 1M, Resistor_SMD:R_0805_2012Metric, symbol Device:R
- added R5, R6: 5.11k, Resistor_SMD:R_0805_2012Metric, symbol Device:R
Connections:
- net GND: now also J2.A1 (GND), J2.A12 (GND), J2.B1 (GND), J2.B12 (GND), R10.1, R5.1, R6.1, R8.1, R9.1
- net at J3.5 (Shield): now also R10.2
- new net: J2.A5 (CC1), R6.2
- new net: J2.B5 (CC2), R5.2
- new net: J2.S1 (SHIELD), R8.2
- new net: J1.5 (Shield), R9.2
- new net +5V: J1.1 (VBUS), J1.2 (D-), J1.3 (D+), J1.4 (GND), J2.A4 (VBUS), J2.A9 (VBUS), J2.B4 (VBUS), J2.B9 (VBUS)
Other:
- moved on the sheet: J3

Commit message: update
Parts:
- added J4, J5: USB_C_Receptacle_USB2.0_16P, Connector_USB:USB_C_Receptacle_G-Switch_GT-USB-7010ASV, symbol Connector:USB_C_Receptacle_USB2.0_16P
- added J6: USB_B_Micro, Connector_USB:USB_Micro-AB_Molex_47590-0001, symbol Connector:USB_B_Micro
- added R11, R12, R7: 1M, Resistor_SMD:R_0805_2012Metric, symbol Device:R
Connections:
- net +5V: now also J4.A1 (GND), J4.A12 (GND), J4.A4 (VBUS), J4.A6 (D+), J4.A7 (D-), J4.A9 (VBUS), J4.B1 (GND), J4.B12 (GND), J4.B4 (VBUS), J4.B6 (D+), J4.B7 (D-), J4.B9 (VBUS)
- net GND: now also R11.1, R12.1, R7.1
- net at D1.2 (A), J3.1 (VBUS): now also J5.A4 (VBUS), J5.A9 (VBUS), J5.B4 (VBUS), J5.B9 (VBUS), J6.1 (VBUS)
- net at D3.2 (A), J3.2 (D-): now also J5.A7 (D-), J5.B7 (D-), J6.2 (D-)
- net at D2.2 (A), J3.3 (D+): now also J5.A6 (D+), J5.B6 (D+), J6.3 (D+)
- net at D4.2 (A), J3.4 (GND): now also J5.A1 (GND), J5.A12 (GND), J5.B1 (GND), J5.B12 (GND), J6.5 (GND)
- new net: J6.6 (Shield), R12.2
- new net: J5.S1 (SHIELD), R7.2
- new net: J4.S1 (SHIELD), R11.2
