File: USB tester/USB tester.kicad_pcb (KiCad board)
At the start: 2 copper layers, 79.5 x 62 mm, 16 parts, among them J1 USB_A, J2 USB_C_Receptacle_USB2.0_16P, J3 USB_A

Commit message: update
Parts:
- added J4: USB_C_Receptacle_USB2.0_16P, Connector_USB:USB_C_Receptacle_G-Switch_GT-USB-7010ASV, F.Cu at (32.0, 109.5)
- added J5: USB_C_Receptacle_USB2.0_16P, Connector_USB:USB_C_Receptacle_G-Switch_GT-USB-7010ASV, F.Cu at (32.0, 54.5)
- added J6: USB_B_Micro, Connector_USB:USB_Micro-AB_Molex_47590-0001, F.Cu at (82.3, 53.5)
- added R11: 1M, Resistor_SMD:R_0805_2012Metric, F.Cu at (40.0, 105.6)
- added R12: 1M, Resistor_SMD:R_0805_2012Metric, F.Cu at (86.7, 48.9)
- added R7: 1M, Resistor_SMD:R_0805_2012Metric, F.Cu at (41.0, 58.9)
Routing:
- net GND: track 0.00 -> 76.3 mm
- net +5V: track 0.00 -> 7.00 mm
- net Net-(J2-CC2): track 0.00 -> 4.88 mm
- net Net-(J2-CC1): track 0.00 -> 4.81 mm
- net Net-(J1-Shield): track 0.00 -> 3.82 mm
- net Net-(J4-SHIELD): track 0.00 -> 3.73 mm
- net Net-(J2-SHIELD): track 0.00 -> 2.37 mm

Commit message: update
Parts:
- moved R12 14.3 mm to (75.0, 57.1), turned to 90 degrees
- turned D1 to 180 degrees
- turned D2 to 180 degrees
- turned D3 to 180 degrees
- turned D4 to 180 degrees
Routing:
- net GND: track 76.3 -> 154.2 mm
- net +5V: track 7.00 -> 75.4 mm
- net Net-(J4-SHIELD): track 3.73 -> 28.3 mm
- net Net-(J5-SHIELD): track 0.00 -> 21.9 mm
- net Net-(J1-Shield): track 3.82 -> 25.1 mm
- net Net-(J6-Shield): track 0.00 -> 19.1 mm
- net Net-(J3-Shield): track 0.00 -> 17.6 mm
- net Net-(J2-SHIELD): track 2.37 -> 15.2 mm
- net Net-(D4-K): track 0.00 -> 2.73 mm
- net Net-(D3-K): track 0.00 -> 2.71 mm
- net Net-(D1-K): track 0.00 -> 2.70 mm
- net Net-(D2-K): track 0.00 -> 2.69 mm

Commit message: update
Routing:
- net Net-(D4-A): track 0.00 -> 113.8 mm, vias 0 -> 4
- net Net-(D2-A): track 0.00 -> 105.6 mm, vias 0 -> 4
- net Net-(D3-A): track 0.00 -> 101.2 mm, vias 0 -> 2
- net Net-(D1-A): track 0.00 -> 84.7 mm, vias 0 -> 4
- net unconnected-(J6-ID-Pad4): track 0.00 -> 2.86 mm, vias 0 -> 1
